Commit message: Update tyrion_ouster.urdf

File: tyrion_ouster.urdf (robot description, URDF)
Before this commit: robot tyrion, 2 links, 1 joints
Links:
- link base_link_inertia: geometry collision box size=0.9 0.9 0.40; visual mesh filename=tyrion_light.dae scale=1 1 1

Commit message: Update tyrion_ouster.urdf

File: tyrion_ouster.urdf (robot description, URDF)
Before this commit: robot tyrion, 2 links, 1 joints
Links:
- link base_link_inertia: geometry collision box size=0.9 0.9 0.40; visual mesh filename=https://github.com/JBesCar/Tyrion_urdf/blob/main/tyrion_lig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 scale=1 1 1
