Commit message: Update tyrion_ouster.urdf

File: rotors_description/urdf/tyrion_ouster.urdf (robot description, URDF)
Before this commit: robot tyrion, 2 links, 1 joints
Links:
- link base_link_inertia: geometry collision box size=0.9 0.9 0.40; visual mesh filename=package://rotors_description/meshes/tyrion_light.dae scale=1 1 1

Commit message: Update tyrion_ouster.urdf

File: rotors_description/urdf/tyrion_ouster.urdf (robot description, URDF)
Before this commit: robot tyrion, 2 links, 1 joints
Links:
- link base_link_inertia: geometry collision box size=0.9 0.9 0.40; visual mesh filename=package://rotors_description/meshes/tyrion.stl scale=1 1 1

Commit message: Update tyrion_ouster.urdf

File: rotors_description/urdf/tyrion_ouster.urdf (robot description, URDF)
Before this commit: robot tyrion, 2 links, 1 joints
Links:
- link base_link_inertia: geometry collision box size=0.9 0.9 0.40; visual mesh filename=package://rotors_description/meshes/tyrion_light.dae scale=0.01 0.01 0.01
